Commit message: Make meshes accessible via RVIZ2 before: Cannot find them with absolute path

File: urdf/sensors/raspberry_pi_camera_2_1.xacro (robot description, xacro)
@@ -11,5 +11,5 @@
                 <origin rpy="0 1.57 0" xyz="0 0 0.0"/>
                 <geometry>
-                    <mesh filename="$(find br_description)/meshes/sensors/raspberry_pi_camera_2_1.stl" scale="1e-3 1e-3 1e-3"/>
+                    <mesh filename="file://$(find br_description)/meshes/sensors/raspberry_pi_camera_2_1.stl" scale="1e-3 1e-3 1e-3"/>
                 </geometry>
             </visual>

File: urdf/sensors/rplidar_a1m8.xacro (robot description, xacro)
@@ -11,5 +11,5 @@
                 <origin rpy="1.57 0 3.14" xyz="0 0 0.0"/>
                 <geometry>
-                    <mesh filename="$(find br_description)/meshes/sensors/rplidar_a1m8.stl" scale="1e-3 1e-3 1e-3"/>
+                    <mesh filename="file://$(find br_description)/meshes/sensors/rplidar_a1m8.stl" scale="1e-3 1e-3 1e-3"/>
                 </geometry>
             </visual>
