Commit message: Make IMU box smaller 1x1x1 cm

File: urdf/sensors/imu.xacro (robot description, xacro)
@@ -9,13 +9,13 @@
             <xacro:dummy_inertia/>
             <visual>
-                <origin rpy="0 0 0" xyz="0 0 0.025"/>
+                <origin rpy="0 0 0" xyz="0 0 0.005"/>
                 <geometry>
-                    <box size="0.05 0.05 0.05"/>
+                    <box size="0.01 0.01 0.01"/>
                 </geometry>
             </visual>
             <collision>
-                <origin rpy="0 0 0" xyz="0 0 0.025"/>
+                <origin rpy="0 0 0" xyz="0 0 0.005"/>
                 <geometry>
-                    <box size="0.05 0.05 0.05"/>
+                    <box size="0.01 0.01 0.01"/>
                 </geometry>
             </collision>
@@ -24,5 +24,5 @@
             <parent link="${prefix}base_link"/>
             <child link="${prefix}sensor_link"/>
-            <origin xyz="0 0 0.025"/>
+            <origin xyz="0 0 0.005"/>
         </joint>
         <link name="${prefix}sensor_link">

Commit message: Change noise-behavior of Lidar + Imu gazebo models

File: urdf/sensors/imu.xacro (robot description, xacro)
@@ -1,4 +1,4 @@
 <robot xmlns:xacro="http://www.ros.org/wiki/xacro">
-    <xacro:macro name="imu" params="*origin sim sim_noise:=0.001 sim_imu_topic:='/imu/data' sim_rate:=100 parent prefix:='imu_'">
+    <xacro:macro name="imu" params="*origin sim sim_noise:=0.1 sim_imu_topic:='/imu/data' sim_rate:=100 parent prefix:='imu_'">
         <joint name="${parent}_to_${prefix}base_link" type="fixed">
             <parent link="${parent}"/>
@@ -47,5 +47,5 @@
                         <noise type="gaussian">
                             <mean>0.0</mean>
-                            <stddev>2e-4</stddev>
+                            <stddev>${sim_noise}</stddev>
                             <bias_mean>0.0000075</bias_mean>
                             <bias_stddev>0.0000008</bias_stddev>
@@ -55,5 +55,5 @@
                         <noise type="gaussian">
                             <mean>0.0</mean>
-                            <stddev>2e-4</stddev>
+                            <stddev>${sim_noise}</stddev>
                             <bias_mean>0.0000075</bias_mean>
                             <bias_stddev>0.0000008</bias_stddev>
@@ -63,5 +63,5 @@
                         <noise type="gaussian">
                             <mean>0.0</mean>
-                            <stddev>2e-4</stddev>
+                            <stddev>${sim_noise}</stddev>
                             <bias_mean>0.0000075</bias_mean>
                             <bias_stddev>0.0000008</bias_stddev>
@@ -73,5 +73,5 @@
                         <noise type="gaussian">
                             <mean>0.0</mean>
-                            <stddev>1.7e-2</stddev>
+                            <stddev>${10 * sim_noise}</stddev>
                             <bias_mean>0.1</bias_mean>
                             <bias_stddev>0.001</bias_stddev>
@@ -81,5 +81,5 @@
                         <noise type="gaussian">
                             <mean>0.0</mean>
-                            <stddev>1.7e-2</stddev>
+                            <stddev>${10 * sim_noise}</stddev>
                             <bias_mean>0.1</bias_mean>
                             <bias_stddev>0.001</bias_stddev>
@@ -89,5 +89,5 @@
                         <noise type="gaussian">
                             <mean>0.0</mean>
-                            <stddev>1.7e-2</stddev>
+                            <stddev>${10 * sim_noise}</stddev>
                             <bias_mean>0.1</bias_mean>
                             <bias_stddev>0.001</bias_stddev>

File: urdf/sensors/rplidar_a1m8.xacro (robot description, xacro)
@@ -1,4 +1,4 @@
 <robot xmlns:xacro="http://www.ros.org/wiki/xacro">
-    <xacro:macro name="rplidar_a1m8" params="*origin sim sim_noise:=0.001 sim_lidar_topic:='/lidar/scan' sim_rate:=30 parent prefix:='lidar_'">
+    <xacro:macro name="rplidar_a1m8" params="*origin sim sim_noise:=0.01 sim_lidar_topic:='/lidar/scan' sim_rate:=30 parent prefix:='lidar_'">
         <joint name="${parent}_to_${prefix}base_link" type="fixed">
             <parent link="${parent}"/>
