Commit message: Add dummy inertias

File: urdf/budget_roomba.urdf.xacro (robot description, xacro)
@@ -1,4 +1,10 @@
 <?xml version="1.0"?>
-<robot name="myfirst">
+<robot name="myfirst" xmlns:xacro="http://www.ros.org/wiki/xacro">
+  <xacro:macro name="dummy_inertia">
+    <inertial>
+      <mass value="0.1"/>
+      <inertia ixx="1e-3" ixy="1e-3" ixz="1e-3" iyy="1e-3" iyz="1e-3" izz="1e-3"/>
+    </inertial>
+  </xacro:macro>
   <link name="base_link">
   </link>
@@ -9,4 +15,5 @@
   </joint>
   <link name="main_body">
+    <xacro:dummy_inertia/>
     <visual>
       <origin rpy="0 0 0" xyz="0 0 0.1"/>
@@ -28,4 +35,5 @@
   </joint>
   <link name="wheel_left">
+    <xacro:dummy_inertia/>
     <visual>
       <origin rpy="0 1.570796327 0" xyz="0.025 0 0 "/>
@@ -47,4 +55,5 @@
   </joint>
   <link name="wheel_right">
+    <xacro:dummy_inertia/>
     <visual>
       <origin rpy="0 1.570796327 0" xyz="0.025 0 0 "/>
@@ -66,4 +75,5 @@
   </joint>
   <link name="back_ball">
+    <xacro:dummy_inertia/>
     <visual>
       <origin rpy="0 0 0" xyz="0 0 -0.05 "/>

Commit message: Modularize URDF with Xacro-Macros

File: urdf/budget_roomba.urdf.xacro (robot description, xacro)
@@ -7,4 +7,5 @@
     </inertial>
   </xacro:macro>
+  <xacro:include filename="$(find br_description)/urdf/motion/diffdrive.xacro" />
   <link name="base_link">
   </link>
@@ -49,9 +50,5 @@
     </collision>
   </link>
-  <joint name="main_body_to_wheel_right" type="continuous">
-    <parent link="main_body"/>
-    <child link="wheel_right"/>
-    <origin xyz="0.2 -0.30 0.0" rpy="0 0 -1.570796327"/>
-  </joint>
+  <xacro:diffdrive sim="$(arg sim)"/>
   <link name="wheel_right">
     <xacro:dummy_inertia/>

Commit message: Add sensor models

File: urdf/budget_roomba.urdf.xacro (robot description, xacro)
@@ -1,11 +1,16 @@
 <?xml version="1.0"?>
-<robot name="myfirst" xmlns:xacro="http://www.ros.org/wiki/xacro">
+<robot name="budget_roomba" xmlns:xacro="http://www.ros.org/wiki/xacro">
   <xacro:macro name="dummy_inertia">
     <inertial>
+      <origin xyz="0 0 0.0" rpy="0 0 0"/>
       <mass value="0.1"/>
-      <inertia ixx="1e-3" ixy="1e-3" ixz="1e-3" iyy="1e-3" iyz="1e-3" izz="1e-3"/>
+      <inertia ixx="1e-2" ixy="0" ixz="0" iyy="1e-2" iyz="0" izz="1e-2"/>
     </inertial>
   </xacro:macro>
   <xacro:include filename="$(find br_description)/urdf/motion/diffdrive.xacro" />
+  <xacro:include filename="$(find br_description)/urdf/sensors/imu.xacro" />
+  <xacro:include filename="$(find br_description)/urdf/sensors/raspberry_pi_camera_2_1.xacro" />
+  <xacro:include filename="$(find br_description)/urdf/sensors/rplidar_a1m8.xacro" />
+  <xacro:arg name="sim" default="true"/>
   <link name="base_link">
   </link>
@@ -18,5 +23,5 @@
     <xacro:dummy_inertia/>
     <visual>
-      <origin rpy="0 0 0" xyz="0 0 0.1"/>
+      <origin rpy="0 0 0" xyz="-0.2 0 0.1"/>
       <geometry>
         <cylinder length="0.2" radius="0.3"/>
@@ -24,5 +29,5 @@
     </visual>
     <collision>
-      <origin rpy="0 0 0" xyz="0 0 0.1"/>
+      <origin rpy="0 0 0" xyz="-0.2 0 0.1"/>
       <geometry>
         <cylinder length="0.2" radius="0.3"/>
@@ -30,47 +35,15 @@
     </collision>
   </link>
-  <joint name="main_body_to_wheel_left" type="continuous">
-    <parent link="main_body"/>
-    <child link="wheel_left"/>
-    <origin xyz="0.2 0.30 0.0" rpy="0 0 1.570796327"/>
-  </joint>
-  <link name="wheel_left">
-    <xacro:dummy_inertia/>
-    <visual>
-      <origin rpy="0 1.570796327 0" xyz="0.025 0 0 "/>
-      <geometry>
-        <cylinder length="0.05" radius="0.1"/>
-      </geometry>
-    </visual>
-    <collision>
-      <origin rpy="0 1.570796327 0" xyz="0.025 0 0 "/>
-      <geometry>
-        <cylinder length="0.05" radius="0.1"/>
-      </geometry>
-    </collision>
-  </link>
-  <xacro:diffdrive sim="$(arg sim)"/>
-  <link name="wheel_right">
-    <xacro:dummy_inertia/>
-    <visual>
-      <origin rpy="0 1.570796327 0" xyz="0.025 0 0 "/>
-      <geometry>
-        <cylinder length="0.05" radius="0.1"/>
-      </geometry>
-    </visual>
-    <collision>
-      <origin rpy="0 1.570796327 0" xyz="0.025 0 0 "/>
-      <geometry>
-        <cylinder length="0.05" radius="0.1"/>
-      </geometry>
-    </collision>
-  </link>
-  <joint name="main_body_to_back_ball" type="continuous">
+  <joint name="main_body_to_back_ball" type="fixed">
     <parent link="main_body"/>
     <child link="back_ball"/>
-    <origin xyz="-0.3 0 0" rpy="0 0 0"/>
+    <origin xyz="-0.5 0 0" rpy="0 0 0"/>
   </joint>
   <link name="back_ball">
-    <xacro:dummy_inertia/>
+    <inertial>
+      <origin xyz="0 0 0.0" rpy="0 0 0"/>
+      <mass value="0.5"/>
+      <inertia ixx="1e-2" ixy="0" ixz="0" iyy="1e-2" iyz="0" izz="1e-2"/>
+    </inertial>
     <visual>
       <origin rpy="0 0 0" xyz="0 0 -0.05 "/>
@@ -86,3 +59,13 @@
     </collision>
   </link>
+  <xacro:diffdrive sim="$(arg sim)"/>
+  <xacro:imu sim="$(arg sim)" sim_noise="0.01" parent="base_link">
+    <origin xyz="0 0 0.3" rpy="0 0 0"/>
+  </xacro:imu>
+  <xacro:raspberry_pi_camera_2_1 sim="$(arg sim)" sim_noise="0.01" parent="base_link">
+    <origin xyz="0 0 0.5" rpy="0 ${1.57 / 2} 0"/>
+  </xacro:raspberry_pi_camera_2_1>
+  <xacro:rplidar_a1m8 sim="$(arg sim)" sim_noise="0.01" parent="base_link">
+    <origin xyz="0 0 0.55" rpy="0 0 0"/>
+  </xacro:rplidar_a1m8>
 </robot>

Commit message: Scale robot down

File: urdf/budget_roomba.urdf.xacro (robot description, xacro)
@@ -4,6 +4,6 @@
     <inertial>
       <origin xyz="0 0 0.0" rpy="0 0 0"/>
-      <mass value="0.1"/>
-      <inertia ixx="1e-2" ixy="0" ixz="0" iyy="1e-2" iyz="0" izz="1e-2"/>
+      <mass value="1e-2"/>
+      <inertia ixx="1e-3" ixy="0" ixz="0" iyy="1e-3" iyz="0" izz="1e-3"/>
     </inertial>
   </xacro:macro>
@@ -18,18 +18,22 @@
     <parent link="base_link"/>
     <child link="main_body"/>
-    <origin xyz="0 0 0.1"/>
+    <origin xyz="0 0 0.05"/>
   </joint>
   <link name="main_body">
-    <xacro:dummy_inertia/>
+    <inertial>
+      <origin xyz="0 0 0.0" rpy="0 0 0"/>
+      <mass value="3"/>
+      <inertia ixx="1e-2" ixy="0" ixz="0" iyy="1e-2" iyz="0" izz="1e-2"/>
+    </inertial>
     <visual>
-      <origin rpy="0 0 0" xyz="-0.2 0 0.1"/>
+      <origin rpy="0 0 0" xyz="-0.1 0 0.15"/>
       <geometry>
-        <cylinder length="0.2" radius="0.3"/>
+        <cylinder length="0.2" radius="0.1"/>
       </geometry>
     </visual>
     <collision>
-      <origin rpy="0 0 0" xyz="-0.2 0 0.1"/>
+      <origin rpy="0 0 0" xyz="-0.1 0 0.15"/>
       <geometry>
-        <cylinder length="0.2" radius="0.3"/>
+        <cylinder length="0.2" radius="0.1"/>
       </geometry>
     </collision>
@@ -38,25 +42,33 @@
     <parent link="main_body"/>
     <child link="back_ball"/>
-    <origin xyz="-0.5 0 0" rpy="0 0 0"/>
+    <origin xyz="-0.3 0 0" rpy="0 0 0"/>
   </joint>
   <link name="back_ball">
     <inertial>
       <origin xyz="0 0 0.0" rpy="0 0 0"/>
-      <mass value="0.5"/>
-      <inertia ixx="1e-2" ixy="0" ixz="0" iyy="1e-2" iyz="0" izz="1e-2"/>
+      <mass value="1e-1"/>
+      <inertia ixx="1e-3" ixy="0" ixz="0" iyy="1e-3" iyz="0" izz="1e-3"/>
     </inertial>
     <visual>
-      <origin rpy="0 0 0" xyz="0 0 -0.05 "/>
+      <origin rpy="0 0 0" xyz="0 0 -0.025 "/>
       <geometry>
-        <sphere radius="0.05"/>
+        <sphere radius="0.025"/>
       </geometry>
     </visual>
     <collision>
-      <origin rpy="0 0 0" xyz="0 0 -0.05 "/>
+      <origin rpy="0 0 0" xyz="0 0 -0.025 "/>
       <geometry>
-        <sphere radius="0.05"/>
+        <sphere radius="0.025"/>
       </geometry>
     </collision>
   </link>
+  <gazebo reference="back_ball">
+        <material>Gazebo/Gold</material>
+        <mu1>0.0</mu1>
+        <mu2>0.0</mu2>
+    </gazebo>
+  <gazebo reference="main_body_to_back_ball">
+    <preserveFixedJoint>true</preserveFixedJoint>
+  </gazebo>
   <xacro:diffdrive sim="$(arg sim)"/>
   <xacro:imu sim="$(arg sim)" sim_noise="0.01" parent="base_link">
@@ -64,8 +76,8 @@
   </xacro:imu>
   <xacro:raspberry_pi_camera_2_1 sim="$(arg sim)" sim_noise="0.01" parent="base_link">
-    <origin xyz="0 0 0.5" rpy="0 ${1.57 / 2} 0"/>
+    <origin xyz="0 0 0.3" rpy="0 ${1.57 / 2} 0"/>
   </xacro:raspberry_pi_camera_2_1>
   <xacro:rplidar_a1m8 sim="$(arg sim)" sim_noise="0.01" parent="base_link">
-    <origin xyz="0 0 0.55" rpy="0 0 0"/>
+    <origin xyz="0 0 0.35" rpy="0 0 0"/>
   </xacro:rplidar_a1m8>
 </robot>

File: urdf/motion/diffdrive.xacro (robot description, xacro)
@@ -4,5 +4,5 @@
     <parent link="main_body"/>
     <child link="wheel_left"/>
-    <origin xyz="0.0 0.30 0.0" rpy="0 0 1.570796327"/>
+    <origin xyz="0.0 0.1 0.0" rpy="0 0 1.570796327"/>
     <calibration rising="0.0"/>
     <dynamics damping="0.0" friction="0.0"/>
@@ -15,5 +15,5 @@
       <origin rpy="0 1.570796327 0" xyz="0.025 0 0 "/>
       <geometry>
-        <cylinder length="0.05" radius="0.1"/>
+        <cylinder length="0.05" radius="0.05"/>
       </geometry>
     </visual>
@@ -21,5 +21,5 @@
       <origin rpy="0 1.570796327 0" xyz="0.025 0 0 "/>
       <geometry>
-        <cylinder length="0.05" radius="0.1"/>
+        <cylinder length="0.05" radius="0.05"/>
       </geometry>
     </collision>
@@ -28,5 +28,5 @@
     <parent link="main_body"/>
     <child link="wheel_right"/>
-    <origin xyz="0.0 -0.30 0.0" rpy="0 0 1.570796327"/>
+    <origin xyz="0.0 -0.1 0.0" rpy="0 0 1.570796327"/>
     <calibration rising="0.0"/>
     <dynamics damping="0.0" friction="0.0"/>
@@ -39,5 +39,5 @@
       <origin rpy="0 1.570796327 0" xyz="-0.025 0 0 "/>
       <geometry>
-        <cylinder length="0.05" radius="0.1"/>
+        <cylinder length="0.05" radius="0.05"/>
       </geometry>
     </visual>
@@ -45,5 +45,5 @@
       <origin rpy="0 1.570796327 0" xyz="-0.025 0 0 "/>
       <geometry>
-        <cylinder length="0.05" radius="0.1"/>
+        <cylinder length="0.05" radius="0.05"/>
       </geometry>
     </collision>
@@ -60,5 +60,5 @@
             <right_joint>main_body_to_wheel_right</right_joint>
             <!-- The distance from the center of one wheel to the other, in meters, defaults to 0.34 m -->
-            <wheel_separation>0.65</wheel_separation>
+            <wheel_separation>0.25</wheel_separation>
             <!-- Diameter of the wheels, in meters, defaults to 0.15 m -->
             <wheel_diameter>0.1</wheel_diameter>
@@ -66,5 +66,5 @@
             <max_wheel_acceleration>1.0</max_wheel_acceleration>
             <!-- Maximum torque which the wheels can produce, in Nm, defaults to 5 Nm -->
-            <max_wheel_torque>1</max_wheel_torque>
+            <max_wheel_torque>5</max_wheel_torque>
             <!-- Topic to receive geometry_msgs/Twist message commands, defaults to `cmd_vel` -->
             <!-- Topic to publish nav_msgs/Odometry messages, defaults to `odom` -->
@@ -83,8 +83,9 @@
         </plugin>
     </gazebo>
-    <gazebo reference="back_ball">
-        <material>Gazebo/Black</material>
-        <mu1>0.0</mu1>
-        <mu2>0.0</mu2>
+    <gazebo reference="wheel_right">
+        <material>Gazebo/Green</material>
+    </gazebo>
+    <gazebo reference="wheel_left">
+        <material>Gazebo/Red</material>
     </gazebo>
   </xacro:if>

Commit message: Improve structure - Launchfile installation to "share" - Introduce launch and xacro arguments

File: urdf/budget_roomba.urdf.xacro (robot description, xacro)
@@ -13,4 +13,5 @@
   <xacro:include filename="$(find br_description)/urdf/sensors/rplidar_a1m8.xacro" />
   <xacro:arg name="sim" default="true"/>
+  <xacro:arg name="ground_truth_tf" default="true"/>
   <link name="base_link">
   </link>
@@ -63,19 +64,23 @@
     </collision>
   </link>
-  <gazebo reference="back_ball">
-        <material>Gazebo/Gold</material>
-        <mu1>0.0</mu1>
-        <mu2>0.0</mu2>
+  <xacro:if value="$(arg sim)">
+    <gazebo reference="back_ball">
+          <material>Gazebo/Gold</material>
+          <mu1>0.0</mu1>
+          <mu2>0.0</mu2>
+      </gazebo>
+    <gazebo reference="main_body_to_back_ball">
+      <preserveFixedJoint>true</preserveFixedJoint>
     </gazebo>
-  <gazebo reference="main_body_to_back_ball">
-    <preserveFixedJoint>true</preserveFixedJoint>
-  </gazebo>
-  <gazebo>
-        <plugin name="budget_roomba_ros_plugin" filename="libbudget_roomba_ros_plugin.so">
-          <world_frame_id>world</world_frame_id>
-          <robot_base_frame_id>base_link</robot_base_frame_id>
-          <ground_truth_tf>true</ground_truth_tf>
-        </plugin>
-    </gazebo>
+    <xacro:if value="$(arg ground_truth_tf)">
+      <gazebo>
+            <plugin name="budget_roomba_ros_plugin" filename="libbudget_roomba_ros_plugin.so">
+              <world_frame_id>world</world_frame_id>
+              <robot_base_frame_id>base_link</robot_base_frame_id>
+              <ground_truth_tf>true</ground_truth_tf>
+            </plugin>
+      </gazebo>
+    </xacro:if>
+  </xacro:if>
   <xacro:diffdrive sim="$(arg sim)"/>
   <xacro:imu sim="$(arg sim)" sim_noise="0.01" parent="base_link">

File: urdf/sensors/rplidar_a1m8.xacro (robot description, xacro)
@@ -1,4 +1,4 @@
 <robot xmlns:xacro="http://www.ros.org/wiki/xacro">
-    <xacro:macro name="rplidar_a1m8" params="*origin sim sim_noise:=0.001 sim_lidar_topic:='/lidar/scan' sim_rate:=100 parent prefix:='lidar_'">
+    <xacro:macro name="rplidar_a1m8" params="*origin sim sim_noise:=0.001 sim_lidar_topic:='/lidar/scan' sim_rate:=30 parent prefix:='lidar_'">
         <joint name="${parent}_to_${prefix}base_link" type="fixed">
             <parent link="${parent}"/>
@@ -11,5 +11,5 @@
                 <origin rpy="1.57 0 3.14" xyz="0 0 0.0"/>
                 <geometry>
-                    <mesh filename="file://$(find br_description)/meshes/sensors/rplidar_a1m8.stl" scale="1e-3 1e-3 1e-3"/>
+                    <mesh filename="$(find br_description)/meshes/sensors/rplidar_a1m8.stl" scale="1e-3 1e-3 1e-3"/>
                 </geometry>
             </visual>

Commit message: Add navigation system-block

File: urdf/budget_roomba.urdf.xacro (robot description, xacro)
@@ -12,4 +12,5 @@
   <xacro:include filename="$(find br_description)/urdf/sensors/raspberry_pi_camera_2_1.xacro" />
   <xacro:include filename="$(find br_description)/urdf/sensors/rplidar_a1m8.xacro" />
+  <xacro:include filename="$(find br_description)/urdf/sensors/nav_unit.xacro" />
   <xacro:arg name="sim" default="true"/>
   <xacro:arg name="ground_truth_tf" default="false"/>
@@ -28,20 +29,20 @@
     </inertial>
     <visual>
-      <origin rpy="0 0 0" xyz="-0.1 0 0.15"/>
+      <origin rpy="0 0 0" xyz="-0.055 0 0.13"/>
       <geometry>
-        <cylinder length="0.2" radius="0.1"/>
+        <box size="0.3 0.2 0.2"/>
       </geometry>
     </visual>
     <collision>
-      <origin rpy="0 0 0" xyz="-0.1 0 0.15"/>
+      <origin rpy="0 0 0" xyz="-0.055 0 0.13"/>
       <geometry>
-        <cylinder length="0.2" radius="0.1"/>
+        <box size="0.3 0.2 0.2"/>
       </geometry>
     </collision>
   </link>
   <joint name="main_body_to_back_ball" type="fixed">
-    <parent link="main_body"/>
+    <parent link="base_link"/>
     <child link="back_ball"/>
-    <origin xyz="-0.3 0 0" rpy="0 0 0"/>
+    <origin xyz="-0.205 0 0" rpy="0 0 0"/>
   </joint>
   <link name="back_ball">
@@ -52,13 +53,13 @@
     </inertial>
     <visual>
-      <origin rpy="0 0 0" xyz="0 0 -0.025 "/>
+      <origin rpy="0 0 0" xyz="0 0 0.01 "/>
       <geometry>
-        <sphere radius="0.025"/>
+        <sphere radius="0.01"/>
       </geometry>
     </visual>
     <collision>
-      <origin rpy="0 0 0" xyz="0 0 -0.025 "/>
+      <origin rpy="0 0 0" xyz="0 0 0.01 "/>
       <geometry>
-        <sphere radius="0.025"/>
+        <sphere radius="0.01"/>
       </geometry>
     </collision>
@@ -83,13 +84,20 @@
     </xacro:if>
   </xacro:if>
-  <xacro:diffdrive sim="$(arg sim)"/>
-  <xacro:imu sim="$(arg sim)" sim_noise="0.01" parent="base_link">
-    <origin xyz="0 0 0.3" rpy="0 0 0"/>
-  </xacro:imu>
-  <xacro:raspberry_pi_camera_2_1 sim="$(arg sim)" sim_noise="0.01" parent="base_link">
-    <origin xyz="0 0 0.3" rpy="0 ${1.57 / 2} 0"/>
-  </xacro:raspberry_pi_camera_2_1>
-  <xacro:rplidar_a1m8 sim="$(arg sim)" sim_noise="0.01" parent="base_link">
-    <origin xyz="0 0 0.35" rpy="0 0 0"/>
-  </xacro:rplidar_a1m8>
+  <xacro:if value="$(arg sim)">
+    <xacro:diffdrive sim="$(arg sim)"/>
+    <xacro:imu sim="$(arg sim)" sim_noise="0.01" parent="base_link">
+      <origin xyz="0 0 0.3" rpy="0 0 0"/>
+    </xacro:imu>
+    <xacro:raspberry_pi_camera_2_1 sim="$(arg sim)" sim_noise="0.01" parent="base_link">
+      <origin xyz="0 0 0.3" rpy="0 ${1.57 / 2} 0"/>
+    </xacro:raspberry_pi_camera_2_1>
+    <xacro:rplidar_a1m8 sim="$(arg sim)" sim_noise="0.01" parent="base_link">
+      <origin xyz="0 0 0.35" rpy="0 0 0"/>
+    </xacro:rplidar_a1m8>
+  </xacro:if>
+  <xacro:unless value="$(arg sim)">
+    <xacro:nav_unit parent="base_link">
+      <origin xyz="-0.18 0 0.235" rpy="0 0 3.14"/>
+    </xacro:nav_unit>
+  </xacro:unless>
 </robot>
